File: cal_switching.sch (KiCad schematic (older format))
At the start: 2 parts, among them U20 TMUX6111PWR, U21 TMUX6111PWR

Commit message: updates to schematic for alternate part #s
Parts:
- U21: Alternate2 Manf# TMUX6113PWR -> DG412CUE+
Changed lines of the file:
@@
 F 4 "TMUX6111PWR" H 5550 5150 50  0001 C CNN "Manf#"
 F 5 "TMUX6112PWR" H 5550 5150 50  0001 C CNN "Alternate Manf#"
-F 6 "TMUX6113PWR" H 5550 5150 50  0001 C CNN "Alternate2 Manf#"
+F 6 "DG412CUE+" H 5550 5150 50  0001 C CNN "Alternate2 Manf#"
 	1    5550 5150
 	1    0    0    -1
@@
 TMUX6111: Logic 0 closes switch\nTMUX6112: Logic 1 closes switch
 $Comp
-L power:+3.3V #PWR?
+L power:+3.3V #PWR0208
 U 1 1 6263D73F
 P 4750 5950
-F 0 "#PWR?" H 4750 5800 50  0001 C CNN
+F 0 "#PWR0208" H 4750 5800 50  0001 C CNN
 F 1 "+3.3V" H 4765 6123 50  0000 C CNN
 F 2 "" H 4750 5950 50  0001 C CNN
@@
 Pin12 is Vlogic for alternate part DG412CUE+
 $Comp
-L power:+3.3V #PWR?
+L power:+3.3V #PWR0209
 U 1 1 62642C9C
 P 4700 2750
-F 0 "#PWR?" H 4700 2600 50  0001 C CNN
+F 0 "#PWR0209" H 4700 2600 50  0001 C CNN
 F 1 "+3.3V" H 4715 2923 50  0000 C CNN
 F 2 "" H 4700 2750 50  0001 C CNN
@@
 Wire Wire Line
 	4700 2800 5000 2800
+Text Notes 4200 3050 0    50   ~ 0
+Pin12 is Vlogic for alternate part DG412CUE+
 Wire Bus Line
 	4450 1700 4450 2750
 Wire Bus Line
 	4400 4850 4400 5900
-Text Notes 4200 3050 0    50   ~ 0
-Pin12 is Vlogic for alternate part DG412CUE+
 $EndSCHEMATC
