File: compensation_switching.sch (KiCad schematic (older format))
At the start: 5 parts, among them U16 TMUX6111PWR

Commit message: gerbers, BOM and fabrication files sent to PCBway
Parts:
- C12: Alternate Manf# (none) -> CL10C332JB8NNNC; Alternative Manf# CL10C332JB8NNNC -> (none)
Changed lines of the file:
@@
 F 3 "~" H 6600 4200 50  0001 C CNN
 F 4 "CC0603JRNPO9BN332" H 6500 4200 50  0001 C CNN "Manf#"
-F 5 "CL10C332JB8NNNC" H 6500 4200 50  0001 C CNN "Alternative Manf#"
+F 5 "CL10C332JB8NNNC" H 6500 4200 50  0001 C CNN "Alternate Manf#"
 F 6 "5%" H 6500 4200 50  0001 C CNN "Tolerance"
 F 7 "50V" H 6500 4200 50  0001 C CNN "voltage"
@@
 Connection ~ 6950 3800
 $Comp
-L power:+3.3V #PWR?
+L power:+3.3V #PWR0213
 U 1 1 624F74AE
 P 4700 4550
-F 0 "#PWR?" H 4700 4400 50  0001 C CNN
+F 0 "#PWR0213" H 4700 4400 50  0001 C CNN
 F 1 "+3.3V" H 4715 4723 50  0000 C CNN
 F 2 "" H 4700 4550 50  0001 C CNN
